File: Hardware/Production-Rev1/GrrCON-Badge-Rev1.brd (EAGLE design)
At the start: 96.2 x 63.2 mm, 98 parts, among them IC1 ATMEGA16U2AU, IC2 SMARTPRJ_ATMEGA328P-AU, IC3 74LS595D, IC4 74LS595D, IC5 MCP1703CB, Q1 16mhz, SW1 PTS645SMT, X1 USBPCB, Y2 CSTCE16M0V53-R0 16MHZ

Commit message: Fixed missing Power Net, spelling
Fixed Spelling of Arduino on silk and documentation.  Fixed missing
power net to ATMEGA328P processor
Routing:
- net +3V3: track 130.1 -> 142.1 mm, vias 5 -> 7
Other:
- board text added: "Based on the Arduino Uno Rev 3 http://arduino.cc"
- board text removed: "Based on the Ardunio Uno Rev 3 http://arduino.cc"
Changed lines of the file:
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@@
 <layer number="25" name="tNames" color="7" fill="1" visible="yes" active="yes"/>
 <layer number="26" name="bNames" color="7" fill="1" visible="yes" active="yes"/>
-<layer number="27" name="tValues" color="7" fill="1" visible="yes" active="yes"/>
-<layer number="28" name="bValues" color="7" fill="1" visible="yes" active="yes"/>
-<layer number="29" name="tStop" color="2" fill="3" visible="yes" active="yes"/>
-<layer number="30" name="bStop" color="5" fill="6" visible="yes" active="yes"/>
-<layer number="31" name="tCream" color="7" fill="4" visible="yes" active="yes"/>
-<layer number="32" name="bCream" color="7" fill="5" visible="yes" active="yes"/>
-<layer number="33" name="tFinish" color="6" fill="3" visible="yes" active="yes"/>
-<layer number="34" name="bFinish" color="6" fill="6" visible="yes" active="yes"/>
-<layer number="35" name="tGlue" color="7" fill="4" visible="yes" active="yes"/>
-<layer number="36" name="bGlue" color="7" fill="5" visible="yes" active="yes"/>
-<layer number="37" name="tTest" color="7" fill="1" visible="yes" active="yes"/>
-<layer number="38" name="bTest" color="7" fill="1" visible="yes" active="yes"/>
-<layer number="39" name="tKeepout" color="4" fill="11" visible="yes" active="yes"/>
-<layer number="40" name="bKeepout" color="1" fill="11" visible="yes" active="yes"/>
-<layer number="41" name="tRestrict" color="4" fill="10" visible="yes" active="yes"/>
-<layer number="42" name="bRestrict" color="1" fill="10" visible="yes" active="yes"/>
-<layer number="43" name="vRestrict" color="2" fill="10" visible="yes" active="yes"/>
-<layer number="44" name="Drills" color="7" fill="1" visible="yes" active="yes"/>
-<layer number="45" name="Holes" color="7" fill="1" visible="yes" active="yes"/>
-<layer number="46" name="Milling" color="3" fill="1" visible="yes" active="yes"/>
-<layer number="47" name="Measures" color="12" fill="1" visible="yes" active="yes"/>
-<layer number="48" name="Document" color="7" fill="1" visible="yes" active="yes"/>
-<layer number="49" name="ReferenceLC" color="13" fill="1" visible="yes" active="yes"/>
-<layer number="50" name="ReferenceLS" color="12" fill="1" visible="yes" active="yes"/>
-<layer number="51" name="tDocu" color="7" fill="1" visible="yes" active="yes"/>
-<layer number="52" name="bDocu" color="7" fill="1" visible="yes" active="yes"/>
+<layer number="27" name="tValues" color="7" fill="1" visible="no" active="yes"/>
+<layer number="28" name="bValues" color="7" fill="1" visible="no" active="yes"/>
+<layer number="29" name="tStop" color="2" fill="3" visible="no" active="yes"/>
+<layer number="30" name="bStop" color="5" fill="6" visible="no" active="yes"/>
+<layer number="31" name="tCream" color="7" fill="4" visible="no" active="yes"/>
+<layer number="32" name="bCream" color="7" fill="5" visible="no" active="yes"/>
+<layer number="33" name="tFinish" color="6" fill="3" visible="no" active="yes"/>
+<layer number="34" name="bFinish" color="6" fill="6" visible="no" active="yes"/>
+<layer number="35" name="tGlue" color="7" fill="4" visible="no" active="yes"/>
+<layer number="36" name="bGlue" color="7" fill="5" visible="no" active="yes"/>
+<layer number="37" name="tTest" color="7" fill="1" visible="no" active="yes"/>
+<layer number="38" name="bTest" color="7" fill="1" visible="no" active="yes"/>
+<layer number="39" name="tKeepout" color="4" fill="11" visible="no" active="yes"/>
+<layer number="40" name="bKeepout" color="1" fill="11" visible="no" active="yes"/>
+<layer number="41" name="tRestrict" color="4" fill="10" visible="no" active="yes"/>
+<layer number="42" name="bRestrict" color="1" fill="10" visible="no" active="yes"/>
+<layer number="43" name="vRestrict" color="2" fill="10" visible="no" active="yes"/>
+<layer number="44" name="Drills" color="7" fill="1" visible="no" active="yes"/>
+<layer number="45" name="Holes" color="7" fill="1" visible="no" active="yes"/>
+<layer number="46" name="Milling" color="3" fill="1" visible="no" active="yes"/>
+<layer number="47" name="Measures" color="12" fill="1" visible="no" active="yes"/>
+<layer number="48" name="Document" color="7" fill="1" visible="no" active="yes"/>
+<layer number="49" name="ReferenceLC" color="13" fill="1" visible="no" active="yes"/>
+<layer number="50" name="ReferenceLS" color="12" fill="1" visible="no" active="yes"/>
+<layer number="51" name="tDocu" color="7" fill="1" visible="no" active="yes"/>
+<layer number="52" name="bDocu" color="7" fill="1" visible="no" active="yes"/>
 <layer number="91" name="Nets" color="2" fill="1" visible="no" active="no"/>
 <layer number="92" name="Busses" color="1" fill="1" visible="no" active="no"/>
@@
 and human stupidity</text>
 <text x="28.6004" y="12.4206" size="1.016" layer="16" font="vector" ratio="12" rot="MR0">Stay Alert, Stay Alive</text>
-<text x="10.4394" y="39.3954" size="0.8128" layer="26" font="vector" rot="SMR270">Based on the Ardunio Uno Rev 3
+<text x="10.4394" y="39.3954" size="0.8128" layer="26" font="vector" rot="SMR270">Based on the Arduino Uno Rev 3
 http://arduino.cc
 </text>
@@
 <wire x1="29.6164" y1="48.2092" x2="29.6164" y2="47.625" width="0.3048" layer="16"/>
 <wire x1="39.4462" y1="35.941" x2="44.7548" y2="35.941" width="0.8128" layer="16"/>
-<wire x1="44.7548" y1="35.941" x2="47.498" y2="33.9598" width="0.8128" layer="16"/>
+<wire x1="44.7548" y1="35.941" x2="47.3282875" y2="34.08236875" width="0.8128" layer="16"/>
+<wire x1="47.3282875" y1="34.08236875" x2="47.498" y2="33.9598" width="0.8128" layer="16"/>
 <wire x1="47.498" y1="33.9598" x2="47.498" y2="30.0736" width="0.8128" layer="16"/>
 <wire x1="47.498" y1="30.0736" x2="49.4665" y2="28.5877" width="0.8128" layer="16"/>
 <wire x1="38.4556" y1="34.9504" x2="39.4462" y2="35.941" width="0.8128" layer="16"/>
-<wire x1="59.1185" y1="28.5877" x2="49.4665" y2="28.5877" width="0.8128" layer="16"/>
+<wire x1="59.1185" y1="28.5877" x2="50.7746" y2="28.5877" width="0.8128" layer="16"/>
+<wire x1="50.7746" y1="28.5877" x2="49.4665" y2="28.5877" width="0.8128" layer="16"/>
 <wire x1="39.4462" y1="35.941" x2="40.0812" y2="35.9664" width="0.8128" layer="16"/>
 <wire x1="40.0812" y1="35.9664" x2="40.1066" y2="42.4688" width="0.8128" layer="16"/>
@@
 <contactref element="C6" pad="2"/>
 <wire x1="54.7306" y1="40.047" x2="54.6964" y2="40.0812" width="0.6096" layer="1"/>
-<wire x1="55.2894" y1="36.6522" x2="55.2894" y2="33.2422" width="0.4064" layer="1"/>
-<wire x1="55.2894" y1="33.2422" x2="52.8828" y2="30.8356" width="0.4064" layer="1"/>
-<wire x1="52.8828" y1="30.8356" x2="52.8828" y2="28.0736" width="0.4064" layer="1"/>
 <wire x1="52.8828" y1="28.0736" x2="52.8894" y2="28.067" width="0.6096" layer="1"/>
 <contactref element="IC2" pad="6"/>
 <wire x1="53.6894" y1="36.6522" x2="53.6894" y2="37.7636" width="0.4064" layer="1"/>
 <wire x1="53.6894" y1="37.7636" x2="54.4576" y2="38.5318" width="0.4064" layer="1"/>
-<wire x1="54.4576" y1="38.5318" x2="54.4576" y2="39.8424" width="0.4064" layer="1"/>
-<wire x1="54.4576" y1="39.8424" x2="54.6964" y2="40.0812" width="0.4064" layer="1"/>
 <wire x1="55.2894" y1="36.6522" x2="55.2894" y2="37.7" width="0.4064" layer="1"/>
 <wire x1="55.2894" y1="37.7" x2="54.4576" y2="38.5318" width="0.4064" layer="1"/>
-<wire x1="49.4665" y1="28.5877" x2="52.8828" y2="28.0736" width="0" layer="19" extent="1-16"/>
+<wire x1="54.4576" y1="39.8424" x2="55.5092" y2="39.8424" width="0.8128" layer="1"/>
+<wire x1="55.5092" y1="39.8424" x2="56.3626" y2="38.989" width="0.8128" layer="1"/>
+<via x="56.3626" y="38.989" extent="1-16" drill="0.7" diameter="1.4224" shape="octagon"/>
+<wire x1="54.4576" y1="38.5318" x2="54.4576" y2="39.8424" width="0.8128" layer="1"/>
+<wire x1="54.4576" y1="39.8424" x2="54.6964" y2="40.0812" width="0.8128" layer="1"/>
+<wire x1="56.3626" y1="38.989" x2="56.3626" y2="38.0746" width="0.8128" layer="16"/>
+<wire x1="56.3626" y1="38.0746" x2="55.2196" y2="36.9316" width="0.8128" layer="16"/>
+<wire x1="55.2196" y1="36.9316" x2="55.2196" y2="34.0868" width="0.8128" layer="16"/>
+<wire x1="55.2196" y1="34.0868" x2="54.229" y2="33.0962" width="0.8128" layer="16"/>
+<wire x1="54.229" y1="33.0962" x2="50.4952" y2="33.0962" width="0.8128" layer="16"/>
+<wire x1="50.4952" y1="33.0962" x2="49.6316" y2="33.9598" width="0.8128" layer="16"/>
+<wire x1="49.6316" y1="33.9598" x2="47.498" y2="33.9598" width="0.8128" layer="16"/>
+<wire x1="52.8828" y1="28.0736" x2="52.8828" y2="27.1272" width="0.4064" layer="1"/>
+<wire x1="52.8828" y1="27.1272" x2="52.0954" y2="26.3398" width="0.4064" layer="1"/>
+<wire x1="52.0954" y1="26.3398" x2="51.1302" y2="26.3144" width="0.4064" layer="1"/>
+<via x="51.1302" y="26.3144" extent="1-16" drill="0.7" diameter="1.4224" shape="octagon"/>
+<wire x1="51.1302" y1="26.3144" x2="51.1048" y2="28.2575" width="0.4064" layer="16"/>
+<wire x1="51.1048" y1="28.2575" x2="50.7746" y2="28.5877" width="0.4064" layer="16"/>
 </signal>
 <signal name="N$3">
