File: Hardware/Production-Rev1/GrrCON-Badge-Rev1.sch (EAGLE design)
At the start: 98 parts, among them IC1 ATMEGA16U2AU, IC2 SMARTPRJ_ATMEGA328P-AU, IC3 74LS595D, IC4 74LS595D, IC5 MCP1703CB, Q1 16mhz, SW1 PTS645SMT, X1 USBPCB, Y2 CSTCE16M0V53-R0 16MHZ

Commit message: Fixed missing Power Net, spelling
Fixed Spelling of Arduino on silk and documentation.  Fixed missing
power net to ATMEGA328P processor
Other:
- note added: "Based on the Arduino Uno Rev 3, licensed under the Creative Commons Attribution Share-Alike license. http://arduino.cc Designed for GrrCON by GR Makers. http://grmakers.com/ Board layout by Mark Farver, Twisted Blades LLC http://www.twistedblades.net/"
- note removed: "Based on the Ardunio Uno Rev 3, licensed under the Creative Commons Attribution Share-Alike license. http://arduino.cc Designed for GrrCON by GR Makers. http://grmakers.com/ Board layout by Mark Farver, Twisted Blades LLC http://www.twistedblades.net/"
Changed lines of the file:
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@@
 <text x="68.58" y="251.46" size="12.7" layer="97">GrrCON 2013 Badge</text>
 <text x="2.54" y="-10.16" size="3.81" layer="97"></text>
-<text x="2.54" y="-17.78" size="3.81" layer="97">Based on the Ardunio Uno Rev 3, licensed under the Creative Commons Attribution Share-Alike license.  http://arduino.cc
+<text x="2.54" y="-17.78" size="3.81" layer="97">Based on the Arduino Uno Rev 3, licensed under the Creative Commons Attribution Share-Alike license.  http://arduino.cc
 Designed for GrrCON by GR Makers.  http://grmakers.com/
 Board layout by Mark Farver, Twisted Blades LLC http://www.twistedblades.net/</text>
